Commit message: smplx_to_bumi新增优化约束

File: assets/bumi3/meshes/BUMI(1)_5.26.urdf (robot description, URDF)
Before this commit: robot BUMI_V3.0_260119, 22 links, 21 joints
Joints:
- joint l_arm_roll_joint: limit lower=-1.04 upper=1.4 effort=0 velocity=0 -> lower=-0.14 upper=1.94 effort=0 velocity=0
- joint r_arm_roll_joint: limit lower=-1.4 upper=1.04 effort=0 velocity=0 -> lower=-1.94 upper=0.14 effort=0 velocity=0
- joint waist_yaw_joint: axis 0 0 -1 -> 0 0 1

File: assets/bumi3/meshes/BUMI_V3.0_260119GG.urdf (robot description, URDF)
Before this commit: robot BUMI_V3.0_260119, 22 links, 21 joints
Joints:
- joint l_arm_roll_joint: limit lower=-1.04 upper=1.4 effort=0 velocity=0 -> lower=-0.14 upper=1.94 effort=0 velocity=0
- joint r_arm_roll_joint: limit lower=-1.4 upper=1.04 effort=0 velocity=0 -> lower=-1.94 upper=0.14 effort=0 velocity=0
- joint waist_yaw_joint: axis 0 0 -1 -> 0 0 1
